File: hikebuddy_dhauladhar/base.brd (EAGLE design)
At the start: 75 x 40 mm, 116 parts, among them J1 MF-CON-MICROUSB-RIGHT, J2 GPS Port, J5 SOLDER_PAD_2, J9 47352-1001, U1 LTC3586EUFE-1#PBF, U2 MAX17260SETD+, U3 MF-DSC-SOT233-MMBT3904, U4 MF-DSC-SOT233-MMBT3904, U5 DRV2605LTDGSRQ1, U6 BMX160

Commit message: hikebuddy 10 day optimized test psm board
Parts:
- removed ANT: PRO-OB-440, PRO-OB-440:PRO-OB-440_1
- removed BME280: BME280, BME280:PSON65P250X250X100-8N
- removed C14, C15, C3, C4: 0.1uF, SparkFun-Capacitors:C0603
- removed C17, C19, C36, C37: 4.7uF, SparkFun-Capacitors:C0603
- removed C2: 4.7pF, SparkFun-Capacitors:C0603
- removed C21, C23, C38, C7, C8: 10uF, SparkFun-Capacitors:C0603
- removed C34: 0.47uF, MF_Passives:C0603
- removed C35: 0.1uF, MF_Passives:C0603
- removed C5, C6: 47pF, SparkFun-Capacitors:C0603
- removed C9: 10uF, MF_Passives:C1206
- removed D1: MF-LED-0603-RED, MF_LEDs:LED0603
- removed D4: MF-LED-3228-RGB, MF_LEDs:PLCC4
- removed ESP32-PICO-D4: ESP32-PICO-D4, ESP32-PICO-D4:PQFN50P700X700X104-49N
- removed FLASH, RESET: MF-SW-TACT-4.2MM, MF_Switches:TACT4.2MM
- removed FT231: FT231XS, FT231XS-U:TSSOP20
- removed J4: (no value), SparkFun-Connectors:1X03_LOCK
- removed J5: SOLDER_PAD_2, SparkFun-Connectors:SOLDER_PAD_2
- removed J6, J7: (no value), SparkFun-Connectors:1X01
- removed J8: (no value), SparkFun-Connectors:1X06_LOCK
- removed J9: 47352-1001, 47352-1001:MOLEX_47352-1001
- removed L1: 30Ω/1.8A, SparkFun-Coils:L0603
- removed R1, R12, R13, R14, R2, R30, R31, R32, R33, R34, R35, R36, R43, R5, R6: 10k, SparkFun-Resistors:R0603
- removed R10, R11, R40, R41, R42: 1k, SparkFun-Resistors:R0603
- removed R15, R17, R18, R19: 100, SparkFun-Resistors:R0603
- removed R21: 1K, MF_Passives:R0603
- removed R3, R4: 27, SparkFun-Resistors:R0603
- removed R37, R38: 2K, SparkFun-Resistors:R0603
- removed S1, S2, S3, S4: B3U-3000P, B3U-3000P:SW_B3U-3000P
- removed U$5: 51441-1093, myLib:FH12-10S-0.5SH
- removed U2: MAX17260SETD+, MAX17260SETD_coulomb:SON40P300X300X80-15N
- removed U3, U4: MF-DSC-SOT233-MMBT3904, MF_Discrete_Semiconductor:SOT-23-3
- removed U5: DRV2605LTDGSRQ1, DRV2605LTDGSRQ1:SOP50P490X110-10N
- removed U6: BMX160, BMX160:PQFN50P250X300X100-14N
- removed UBLOX_GPS: CAM-M8C-0, CAM-M8C-0:LCC100P960X1400X210-31N
- C1: value 4.7pF -> 1uF; device SparkFun-Capacitors:C0603 -> MF_Passives:C0603
- C12, C29, C30: value 22uF -> 1uF
- C16, C24, C27, C28: value 10uF -> 1uF
- J2: value GPS Port -> (none); device SparkFun-Connectors:1X06_LOCK -> SparkFun-Connectors:1X05_LOCK
- J3: device SparkFun-Connectors:1X03_LOCK -> SparkFun-Connectors:1X05_LOCK
- R7: value 2K -> 3K
- moved J2 55.8 mm to (15.3, 36.8), turned to 0 degrees
- moved C1 32.3 mm to (8.65, 37.4), turned to 270 degrees
- moved J3 29.1 mm to (15.2, 33.9)
Connections:
- removed net ACCL1: ESP32-PICO-D4.13, J8.6
- removed net ACCL2: ESP32-PICO-D4.12, U6.4
- removed net BAT_ALERT: U2.12
- removed net ESP_EN: C3.2, ESP32-PICO-D4.9, R1.1, RESET.P$1, RESET.P$2, U4.P$3
- removed net ESP_FLASH: ESP32-PICO-D4.23, FLASH.P$1, FLASH.P$2, J4.3, R2.1, U3.P$3
- removed net ESP_RX: ESP32-PICO-D4.40, FT231.20, J6.1, R11.1
- removed net ESP_TX: ESP32-PICO-D4.41, FT231.4, J7.1, R10.1
- removed net GPS_RESET: J2.2, R18.2
- removed net GPS_RX: ESP32-PICO-D4.29, J2.5, R17.2
- removed net GPS_SAFEBOOT: J2.3, R19.2
- removed net GPS_TX: ESP32-PICO-D4.28, J2.4, R15.1
- removed net HAP_EN: ESP32-PICO-D4.11, U5.5
- removed net I2C_SCL: BME280.4, ESP32-PICO-D4.42, J3.2, R37.1, U2.14, U5.2, U6.13
- removed net I2C_SDA: BME280.3, ESP32-PICO-D4.39, J3.3, R38.1, U2.13, U5.3, U6.14
- removed net LCD_CLK: ESP32-PICO-D4.17, J8.5, U$5.SCLK
- removed net LCD_CS: ESP32-PICO-D4.21, J8.3, U$5.SCS
- removed net LCD_MOSI: ESP32-PICO-D4.20, J8.4, U$5.SI
- removed net LED1: ESP32-PICO-D4.18, R40.1
- removed net LED2: ESP32-PICO-D4.15, R41.1
- removed net LED3: ESP32-PICO-D4.14, R42.1
- removed net MAGDRDY: ESP32-PICO-D4.10, U$5.EXTCOMIN
- removed net N$1: C1.1, ESP32-PICO-D4.2, L1.1
- removed net N$17: D1.ANODE, R21.P$1
- removed net N$19: J9.8
- removed net N$2: ANT.2, C1.2, C2.2
- removed net N$28: D4.P$2, R40.2
- removed net N$29: R15.2, UBLOX_GPS.25
- removed net N$3: R5.2, U3.P$1
- removed net N$30: R17.1, UBLOX_GPS.26
- removed net N$32: D4.P$3, R42.2
- removed net N$33: D4.P$4, R41.2
- removed net N$34: UBLOX_GPS.16, UBLOX_GPS.17
- removed net N$37: R18.1, UBLOX_GPS.23
- removed net N$38: R19.1, UBLOX_GPS.24
- removed net N$4: R6.2, U4.P$1
- removed net N$41: C36.1, U5.1
- removed net N$45: J9.1
- removed net N$47: C34.P$2, U2.11
- removed net N$5: C4.1, FT231.13, FT231.14, FT231.3
- removed net N$50: J5.P$2, U5.9
- removed net N$51: J5.P$1, U5.7
- removed net N$6: FT231.12, R3.2
- removed net N$7: FT231.11, R4.2
- removed net N$8: FT231.2, R5.1, U4.P$2
- removed net N$9: FT231.1, R6.1, U3.P$2
- removed net NC0: ESP32-PICO-D4.32
- removed net NC1: ESP32-PICO-D4.33
- removed net NC2: ESP32-PICO-D4.30
- removed net NC3: ESP32-PICO-D4.31
- removed net NC4: ESP32-PICO-D4.25
- removed net NC5: ESP32-PICO-D4.27
- removed net SD_CLK: ESP32-PICO-D4.35, J9.5, R14.1
- removed net SD_CS: ESP32-PICO-D4.34, J9.2, R12.1
- removed net SD_MISO: ESP32-PICO-D4.38, J9.7, R43.1
- removed net SD_MOSI: ESP32-PICO-D4.36, J9.3, R13.1
- removed net SW1: ESP32-PICO-D4.5, R32.1, S1.2
- removed net SW2: ESP32-PICO-D4.6, R33.1, S2.2
- removed net SW3: ESP32-PICO-D4.7, R34.1, S3.2
- removed net SW4: ESP32-PICO-D4.8, R35.1, S4.2
- net 3V3_GPS: now also J3.2; no longer C17.1, J2.6, UBLOX_GPS.1, UBLOX_GPS.9
- net 3V3_SDC: now also J3.5; no longer C14.1, C15.1, J9.4, R12.2, R13.2, R14.2, R43.2
- net D+: no longer C6.1, R4.1
- net D-: no longer C5.1, R3.1
- net EN_GPS: now also J2.2; no longer ESP32-PICO-D4.16, R31.2
- net EN_LCD: now also J2.4; no longer ESP32-PICO-D4.24, R36.2
- net EN_SDC: now also J2.5; no longer ESP32-PICO-D4.22, R30.2
- net GND: now also C1.P$1; no longer ANT.1, BME280.1, BME280.5, BME280.7, C14.2, C15.2, C17.2, C19.1, C2.1, C21.2, C23.2, C3.1, C34.P$1, C35.P$1, C36.2, C37.1, C38.1, C4.2, C5.2, C6.2, C7.2, C8.1, C9.P$2, ESP32-PICO-D4.49, FLASH.P$3, FLASH.P$4, FT231.16, FT231.6, J3.1, J4.1, J8.1, J9.6, J9.S1, J9.S2, J9.S3, J9.S4, L1.2, R30.1, R31.1, R36.1, RESET.P$3, RESET.P$4, S1.1, S2.1, S3.1, S4.1, U$5.VSS, U$5.VSSA, U2.15, U2.8, U2.9, U5.4, U5.8, U6.1, U6.2, U6.3, U6.6, U6.7, UBLOX_GPS.10, UBLOX_GPS.11, UBLOX_GPS.12, UBLOX_GPS.13, UBLOX_GPS.14, UBLOX_GPS.15, UBLOX_GPS.18, UBLOX_GPS.19, UBLOX_GPS.21, UBLOX_GPS.22, UBLOX_GPS.27, UBLOX_GPS.31, UBLOX_GPS.4, UBLOX_GPS.5
- net N$16: no longer D1.CATHODE
- net VCC: now also J2.3; no longer BME280.2, BME280.6, BME280.8, C21.1, C23.1, C38.2, C8.2, D4.P$1, ESP32-PICO-D4.1, ESP32-PICO-D4.19, ESP32-PICO-D4.26, ESP32-PICO-D4.3, ESP32-PICO-D4.37, ESP32-PICO-D4.4, ESP32-PICO-D4.43, ESP32-PICO-D4.46, J4.2, R1.2, R10.2, R11.2, R2.2, R32.2, R33.2, R34.2, R35.2, R37.2, R38.2, U6.12, U6.5, U6.8
- net V_BAT: now also J3.3; no longer C35.P$2, C37.2, U2.1, U2.10, U2.6, U2.7, U5.10, U5.6, UBLOX_GPS.8
- net V_LCD: now also J3.4; no longer C19.2, J8.2, U$5.DISP, U$5.EXTMODE, U$5.VDD, U$5.VDDA
- net V_REG: now also J3.1; no longer R21.P$2
- net V_USB: now also C1.P$2; no longer C7.1, C9.P$1, FT231.15
Routing:
- net GND: track 497.5 -> 123.5 mm, vias 94 -> 14
- net VCC: track 230.8 -> 33.8 mm, vias 18 -> 3
- net 3V3_GPS: track 147.8 -> 19.0 mm, vias 8 -> 3
- net I2C_SDA: track 111.2 -> 0.00 mm, vias 5 -> 0
- net I2C_SCL: track 109.8 -> 0.00 mm, vias 4 -> 0
- net V_BAT: track 119.1 -> 26.6 mm, vias 5 -> 2
- net SW2: track 89.0 -> 0.00 mm, vias 2 -> 0
- net SW4: track 71.6 -> 0.00 mm, vias 3 -> 0
- net GPS_TX: track 70.9 -> 0.00 mm, vias 3 -> 0
- net GPS_RX: track 70.3 -> 0.00 mm, vias 3 -> 0
- net SW1: track 68.1 -> 0.00 mm, vias 4 -> 0
- net ESP_RX: track 68.0 -> 0.00 mm, vias 3 -> 0
- net ESP_FLASH: track 67.4 -> 0.00 mm, vias 5 -> 0
- net ESP_TX: track 64.0 -> 0.00 mm, vias 3 -> 0
- net SW3: track 58.6 -> 0.00 mm, vias 3 -> 0
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- removed copper zone on layer 1, net VCC
- removed copper zone on layer 16, net V_BAT
Other:
- board size 75 x 40 mm -> 27 x 25 mm
- board text added: "BAT"
- board text added: "EN"
- board text added: "GPS"
- board text added: "LCD"
- board text added: "OUT"
- board text added: "REG"
- board text added: "SDC"
- board text removed: "2020 Saurabh Gandhi"
- board text removed: "ESP_RX"
- board text removed: "ESP_TX"
- board text removed: "GPIO/ Flash"
- board text removed: "GPS / UART Extension"
- board text removed: "Hikebuddy 2.0 Dhauladhar"
- board text removed: "I2C Extension"
- board text removed: "IO13"
- board text removed: "IO14"
- board text removed: "IO15"
- board text removed: "IO33"
- board text removed: "LCD / GPIO Extension"
- board text removed: "RESET"
- board text removed: "RX"
- board text removed: "SAFEBOOT"
- board text removed: "SCL"
- board text removed: "SDA"
- board text removed: "TX"
- board text removed: "VCC (LCD)"
- board text removed: "V_GPS (3.3V)"
