File: hikebuddy_dhauladhar/base.sch (EAGLE design)
At the start: 116 parts, among them J1 MF-CON-MICROUSB-RIGHT, J2 GPS Port, J5 SOLDER_PAD_2, J9 47352-1001, U1 LTC3586EUFE-1#PBF, U2 MAX17260SETD+, U3 MF-DSC-SOT233-MMBT3904, U4 MF-DSC-SOT233-MMBT3904, U5 DRV2605LTDGSRQ1, U6 BMX160

Commit message: hikebuddy 10 day optimized test psm board
Parts:
- removed ANT: PRO-OB-440, PRO-OB-440:PRO-OB-440
- removed BME280: BME280, BME280:BME280
- removed C14, C15: 0.1uF, SparkFun-Capacitors:0.1UF-0603-25V-5%
- removed C17: 4.7uF, SparkFun-Capacitors:0.1UF-0603-25V-5%
- removed C19, C36, C37: 4.7uF, SparkFun-Capacitors:4.7UF-0603-6.3V-(10%)
- removed C2: 4.7pF, SparkFun-Capacitors:4.7PF-0603-50V-5%
- removed C21, C23: 10uF, SparkFun-Capacitors:10UF-0603-6.3V-20%
- removed C3, C4: 0.1uF, SparkFun-Capacitors:0.1UF-0603-25V-(+80/-20%)
- removed C34: 0.47uF, MF_Passives:CAPACITOR_NP_0603
- removed C35: 0.1uF, MF_Passives:CAPACITOR_NP_0603
- removed C38, C8: 10uF, SparkFun-Capacitors:4.7PF-0603-50V-5%
- removed C5, C6: 47pF, SparkFun-Capacitors:47PF-0603-50V-5%
- removed C7: 10uF, SparkFun-Capacitors:2.2UF-0603-10V-20%
- removed C9: 10uF, MF_Passives:CAPACITOR_NP_1206
- removed D1: MF-LED-0603-RED, MF_LEDs:LED_SINGLE-0603-RED
- removed D4: MF-LED-3228-RGB, MF_LEDs:LED_RGB_CA_PLCC4
- removed ESP32-PICO-D4: ESP32-PICO-D4, ESP32-PICO-D4:ESP32-PICO-D4
- removed FLASH, RESET: MF-SW-TACT-4.2MM, MF_Switches:TACT_4.2MM
- removed FT231: FT231XS, FT231XS-U:FT231XS-UTSSOP20
- removed J4: (no value), SparkFun-Connectors:CONN_03LOCK
- removed J5: SOLDER_PAD_2, SparkFun-Connectors:SOLDER_PAD_2
- removed J6, J7: (no value), SparkFun-Connectors:CONN_01
- removed J8: (no value), SparkFun-Connectors:CONN_06LOCK
- removed J9: 47352-1001, 47352-1001:47352-1001
- removed L1: 30Ω/1.8A, SparkFun-Coils:FERRITE_BEAD-0603
- removed R1, R12, R13, R14, R2, R30, R31, R32, R33, R34, R35, R36, R43, R5, R6: 10k, SparkFun-Resistors:10KOHM-0603-1/10W-1%
- removed R10, R11, R40, R41, R42: 1k, SparkFun-Resistors:1KOHM-0603-1/10W-1%
- removed R15, R17, R18, R19: 100, SparkFun-Resistors:1KOHM-0603-1/10W-1%
- removed R21: 1K, MF_Passives:RESISTOR_0603
- removed R3, R4: 27, SparkFun-Resistors:27OHM-0603-1/10W-1%
- removed R37, R38: 2K, SparkFun-Resistors:1KOHM-0603-1/10W-1%
- removed S1, S2, S3, S4: B3U-3000P, B3U-3000P:B3U-3000P
- removed U$5: 51441-1093, myLib:LS027B_LCD_SHARPFH12-10S-0.5SH
- removed U2: MAX17260SETD+, MAX17260SETD_coulomb:MAX17260SETD+
- removed U3, U4: MF-DSC-SOT233-MMBT3904, MF_Discrete_Semiconductor:NPN_BJTMMBT3904_SOT-23-3
- removed U5: DRV2605LTDGSRQ1, DRV2605LTDGSRQ1:DRV2605LTDGSRQ1
- removed U6: BMX160, BMX160:BMX160
- removed UBLOX_GPS: CAM-M8C-0, CAM-M8C-0:CAM-M8C-0
- C1: value 4.7pF -> 1uF; device SparkFun-Capacitors:4.7PF-0603-50V-5% -> MF_Passives:CAPACITOR_NP_0603
- C12, C29, C30: value 22uF -> 1uF
- C16, C24, C27, C28: value 10uF -> 1uF
- J2: value GPS Port -> (none); device SparkFun-Connectors:CONN_06LOCK -> SparkFun-Connectors:CONN_05LOCK
- J3: device SparkFun-Connectors:CONN_03LOCK -> SparkFun-Connectors:CONN_05LOCK
- R7: value 2K -> 3K
Connections:
- removed net ACCL1: ESP32-PICO-D4.IO33, J8.6
- removed net ACCL2: ESP32-PICO-D4.IO32, U6.INT1
- removed net BAT_ALERT: U2.ALRT
- removed net ESP_EN: C3.2, ESP32-PICO-D4.EN, R1.1, RESET.P$1, RESET.P$2, U4.COLLECTOR
- removed net ESP_FLASH: ESP32-PICO-D4.IO0, FLASH.P$1, FLASH.P$2, J4.3, R2.1, U3.COLLECTOR
- removed net ESP_RX: ESP32-PICO-D4.U0RXD, FT231.TXD, J6.1, R11.1
- removed net ESP_TX: ESP32-PICO-D4.U0TXD, FT231.RXD, J7.1, R10.1
- removed net GPS_RESET: J2.2, R18.2
- removed net GPS_RX: ESP32-PICO-D4.SD3, J2.5, R17.2
- removed net GPS_SAFEBOOT: J2.3, R19.2
- removed net GPS_TX: ESP32-PICO-D4.SD2, J2.4, R15.1
- removed net HAP_EN: ESP32-PICO-D4.IO35, U5.EN
- removed net I2C_SCL: BME280.SCK, ESP32-PICO-D4.IO21, J3.2, R37.1, U2.SCL, U5.SCL, U6.SCX
- removed net I2C_SDA: BME280.SDI, ESP32-PICO-D4.IO22, J3.3, R38.1, U2.SDA, U5.SDA, U6.SDX
- removed net LCD_CLK: ESP32-PICO-D4.IO14, J8.5, U$5.SCLK
- removed net LCD_CS: ESP32-PICO-D4.IO15, J8.3, U$5.SCS
- removed net LCD_MOSI: ESP32-PICO-D4.IO13, J8.4, U$5.SI
- removed net LED1: ESP32-PICO-D4.IO12, R40.1
- removed net LED2: ESP32-PICO-D4.IO26, R41.1
- removed net LED3: ESP32-PICO-D4.IO25, R42.1
- removed net MAGDRDY: ESP32-PICO-D4.IO34, U$5.EXTCOMIN
- removed net N$1: C1.1, ESP32-PICO-D4.LNA_IN, L1.1
- removed net N$17: D1.ANODE, R21.P$1
- removed net N$19: J9.DATA1
- removed net N$2: ANT.RF_FEED, C1.2, C2.2
- removed net N$28: D4.CATHODE_RED, R40.2
- removed net N$29: R15.2, UBLOX_GPS.TXD/SPI_MISO
- removed net N$3: R5.2, U3.BASE
- removed net N$30: R17.1, UBLOX_GPS.RXD/SPI_MOSI
- removed net N$32: D4.CATHODE_GREEN, R42.2
- removed net N$33: D4.CATHODE_BLUE, R41.2
- removed net N$34: UBLOX_GPS.RF_IN, UBLOX_GPS.RF_OUT
- removed net N$37: R18.1, UBLOX_GPS.RESET_N
- removed net N$38: R19.1, UBLOX_GPS.SAFEBOOT_N
- removed net N$4: R6.2, U4.BASE
- removed net N$41: C36.1, U5.REG
- removed net N$45: J9.DATA2
- removed net N$47: C34.P$2, U2.REG
- removed net N$5: C4.1, FT231.!RESET#, FT231.3V3OUT, FT231.VCCIO
- removed net N$50: J5.2, U5.OUT-
- removed net N$51: J5.1, U5.OUT+
- removed net N$6: FT231.USBDM, R3.2
- removed net N$7: FT231.USBDP, R4.2
- removed net N$8: FT231.!RTS#, R5.1, U4.EMITTER
- removed net N$9: FT231.!DTR#, R6.1, U3.EMITTER
- removed net NC0: ESP32-PICO-D4.SD0
- removed net NC1: ESP32-PICO-D4.SD1
- removed net NC2: ESP32-PICO-D4.CMD
- removed net NC3: ESP32-PICO-D4.CLK
- removed net NC4: ESP32-PICO-D4.IO16
- removed net NC5: ESP32-PICO-D4.IO17
- removed net SD_CLK: ESP32-PICO-D4.IO18, J9.CLK, R14.1
- removed net SD_CS: ESP32-PICO-D4.IO5, J9.CD/DATA3, R12.1
- removed net SD_MISO: ESP32-PICO-D4.IO19, J9.DATA0, R43.1
- removed net SD_MOSI: ESP32-PICO-D4.IO23, J9.CMD, R13.1
- removed net SW1: ESP32-PICO-D4.SENSOR_VP, R32.1, S1.2
- removed net SW2: ESP32-PICO-D4.SENSOR_CAPP, R33.1, S2.2
- removed net SW3: ESP32-PICO-D4.SENSOR_CAPN, R34.1, S3.2
- removed net SW4: ESP32-PICO-D4.SENSOR_VN, R35.1, S4.2
- net 3V3_GPS: now also J3.2; no longer C17.1, J2.6, UBLOX_GPS.VCC, UBLOX_GPS.VCC_IO
- net 3V3_SDC: now also J3.5; no longer C14.1, C15.1, J9.VDD, R12.2, R13.2, R14.2, R43.2
- net D+: no longer C6.1, R4.1
- net D-: no longer C5.1, R3.1
- net EN_GPS: now also J2.2; no longer ESP32-PICO-D4.IO27, R31.2
- net EN_LCD: now also J2.4; no longer ESP32-PICO-D4.IO4, R36.2
- net EN_SDC: now also J2.5; no longer ESP32-PICO-D4.IO2, R30.2
- net GND: now also C1.P$1; no longer ANT.GND, BME280.GND, BME280.SDO, C14.2, C15.2, C17.2, C19.1, C2.1, C21.2, C23.2, C3.1, C34.P$1, C35.P$1, C36.2, C37.1, C38.1, C4.2, C5.2, C6.2, C7.2, C8.1, C9.P$2, ESP32-PICO-D4.GND, FLASH.P$3, FLASH.P$4, FT231.GND, J3.1, J4.1, J8.1, J9.SHIELD, J9.VSS, L1.2, R30.1, R31.1, R36.1, RESET.P$3, RESET.P$4, S1.1, S2.1, S3.1, S4.1, U$5.VSS, U$5.VSSA, U2.CSPL, U2.EP, U2.GND, U5.GND, U5.IN/TRIG, U6.GND, U6.GNDIO, U6.SDO, UBLOX_GPS.GND, UBLOX_GPS.GND-1, UBLOX_GPS.GND-10, UBLOX_GPS.GND-11, UBLOX_GPS.GND-12, UBLOX_GPS.GND-13, UBLOX_GPS.GND-2, UBLOX_GPS.GND-3, UBLOX_GPS.GND-4, UBLOX_GPS.GND-5, UBLOX_GPS.GND-6, UBLOX_GPS.GND-7, UBLOX_GPS.GND-8, UBLOX_GPS.GND-9
- net N$16: no longer D1.CATHODE
- net VCC: now also J2.3; no longer BME280.CSB, BME280.VDD, BME280.VDDIO, C21.1, C23.1, C38.2, C8.2, D4.ANODE, ESP32-PICO-D4.VDD3P3_CPU, ESP32-PICO-D4.VDD3P3_RTC, ESP32-PICO-D4.VDDA, ESP32-PICO-D4.VDDA3P3, ESP32-PICO-D4.VDD_SDIO, J4.2, R1.2, R10.2, R11.2, R2.2, R32.2, R33.2, R34.2, R35.2, R37.2, R38.2, U6.CSB, U6.VDD, U6.VDDIO
- net V_BAT: now also J3.3; no longer C35.P$2, C37.2, U2.BATT, U2.CSN, U2.CSPH, U2.TH, U5.VDD, U5.VDD/NC, UBLOX_GPS.V_BCKP
- net V_LCD: now also J3.4; no longer C19.2, J8.2, U$5.DISP, U$5.EXTMODE, U$5.VDD, U$5.VDDA
- net V_REG: now also J3.1; no longer R21.P$2
- net V_USB: now also C1.P$2; no longer C7.1, C9.P$1, FT231.VCC
