File: hikebuddy_dhauladhar/base.sch (EAGLE design)
At the start: 116 parts, among them J1 MF-CON-MICROUSB-RIGHT, J2 GPS Port, J5 SOLDER_PAD_2, J9 47352-1001, U1 LTC3586EUFE-1#PBF, U2 MAX17260SETD+, U3 MF-DSC-SOT233-MMBT3904, U4 MF-DSC-SOT233-MMBT3904, U5 DRV2605LTDGSRQ1, U6 BMX160

Commit message: fixed power, routed bmx160, changed and routed buttons; cs_v2_non_macrofab
Parts:
- S1, S2, S3, S4: value B3U-3000P -> EVQ-P4HB3B; device B3U-3000P:B3U-3000P -> EVQ-P4HB3B:EVQ-P4HB3B
Connections:
- net GND: now also S1.2, S1.SHIELD, S2.2, S2.SHIELD, S3.2, S3.SHIELD, S4.2, S4.SHIELD; no longer S1.1, S2.1, S3.1, S4.1
- net SW1: now also S1.1; no longer S1.2
- net SW2: now also S4.1; no longer S2.2
- net SW3: now also S3.1; no longer S3.2
- net SW4: now also S2.1; no longer S4.2
Changed lines of the file:
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@@
 <part name="C36" library="SparkFun-Capacitors" deviceset="4.7UF" device="-0603-6.3V-(10%)" package3d_urn="urn:adsk.eagle:package:23616/2" value="4.7uF"/>
 <part name="C37" library="SparkFun-Capacitors" deviceset="4.7UF" device="-0603-6.3V-(10%)" package3d_urn="urn:adsk.eagle:package:23616/2" value="4.7uF"/>
-<part name="S1" library="B3U-3000P" deviceset="B3U-3000P" device="" package3d_urn="urn:adsk.eagle:package:16346045/2" override_package3d_urn="urn:adsk.eagle:package:16346036/2" override_package_urn="urn:adsk.eagle:footprint:16346037/1" override_locally_modified="yes"/>
-<part name="S2" library="B3U-3000P" deviceset="B3U-3000P" device="" package3d_urn="urn:adsk.eagle:package:16346045/2" override_package3d_urn="urn:adsk.eagle:package:16346040/2" override_package_urn="urn:adsk.eagle:footprint:16346041/1" override_locally_modified="yes"/>
-<part name="S3" library="B3U-3000P" deviceset="B3U-3000P" device="" package3d_urn="urn:adsk.eagle:package:16346045/2"/>
-<part name="S4" library="B3U-3000P" deviceset="B3U-3000P" device="" package3d_urn="urn:adsk.eagle:package:16346045/2" override_package3d_urn="urn:adsk.eagle:package:16346042/2" override_package_urn="urn:adsk.eagle:footprint:16346043/1" override_locally_modified="yes"/>
 <part name="GND14" library="supply1" library_urn="urn:adsk.eagle:library:371" deviceset="GND" device=""/>
 <part name="R32" library="SparkFun-Resistors" deviceset="10KOHM" device="-0603-1/10W-1%" package3d_urn="urn:adsk.eagle:package:23555/3" value="10k"/>
@@
 <part name="3V3_ESP5" library="SparkFun-PowerSymbols" library_urn="urn:adsk.eagle:library:530" deviceset="VCC" device="" value="3V3_ESP"/>
 <part name="C21" library="SparkFun-Capacitors" deviceset="10UF" device="-0603-6.3V-20%" package3d_urn="urn:adsk.eagle:package:23616/2" value="10uF"/>
+<part name="S2" library="EVQ-P4HB3B" deviceset="EVQ-P4HB3B" device="" override_package3d_urn="urn:adsk.eagle:package:16346036/2" override_package_urn="urn:adsk.eagle:footprint:16346037/1" override_locally_modified="yes"/>
+<part name="S3" library="EVQ-P4HB3B" deviceset="EVQ-P4HB3B" device="" override_package3d_urn="urn:adsk.eagle:package:16346036/2" override_package_urn="urn:adsk.eagle:footprint:16346037/1" override_locally_modified="yes"/>
+<part name="S4" library="EVQ-P4HB3B" deviceset="EVQ-P4HB3B" device="" override_package3d_urn="urn:adsk.eagle:package:16346036/2" override_package_urn="urn:adsk.eagle:footprint:16346037/1" override_locally_modified="yes"/>
+<part name="S1" library="EVQ-P4HB3B" deviceset="EVQ-P4HB3B" device="" override_package3d_urn="urn:adsk.eagle:package:16346036/2" override_package_urn="urn:adsk.eagle:footprint:16346037/1" override_locally_modified="yes"/>
 </parts>
 <sheets>
@@
 <attribute name="VALUE" x="244.221" y="51.816" size="1.778" layer="96" font="vector" rot="R270"/>
 </instance>
-<instance part="S1" gate="G$1" x="66.04" y="22.86" smashed="yes">
-<attribute name="NAME" x="58.40906875" y="27.947290625" size="2.543640625" layer="95"/>
-<attribute name="VALUE" x="58.40628125" y="15.22628125" size="2.54456875" layer="96"/>
-</instance>
-<instance part="S2" gate="G$1" x="66.04" y="5.08" smashed="yes">
-<attribute name="NAME" x="58.40906875" y="10.167290625" size="2.543640625" layer="95"/>
-<attribute name="VALUE" x="58.40628125" y="-2.55371875" size="2.54456875" layer="96"/>
-</instance>
-<instance part="S3" gate="G$1" x="66.04" y="-12.7" smashed="yes">
-<attribute name="NAME" x="58.40906875" y="-7.612709375" size="2.543640625" layer="95"/>
-<attribute name="VALUE" x="58.40628125" y="-20.33371875" size="2.54456875" layer="96"/>
-</instance>
-<instance part="S4" gate="G$1" x="66.04" y="-30.48" smashed="yes">
-<attribute name="NAME" x="58.40906875" y="-25.392709375" size="2.543640625" layer="95"/>
-<attribute name="VALUE" x="58.40628125" y="-38.11371875" size="2.54456875" layer="96"/>
-</instance>
 <instance part="GND14" gate="1" x="78.74" y="-40.64" smashed="yes">
 <attribute name="VALUE" x="76.2" y="-43.18" size="1.778" layer="96"/>
@@
 <attribute name="NAME" x="405.384" y="112.141" size="1.778" layer="95" font="vector"/>
 <attribute name="VALUE" x="405.384" y="107.061" size="1.778" layer="96" font="vector"/>
+</instance>
+<instance part="S2" gate="G$1" x="68.58" y="-30.48" smashed="yes">
+<attribute name="NAME" x="60.94906875" y="-25.392709375" size="2.543640625" layer="95"/>
+<attribute name="VALUE" x="60.94628125" y="-38.11371875" size="2.54456875" layer="96"/>
+</instance>
+<instance part="S3" gate="G$1" x="68.58" y="-12.7" smashed="yes">
+<attribute name="NAME" x="60.94906875" y="-7.612709375" size="2.543640625" layer="95"/>
+<attribute name="VALUE" x="60.94628125" y="-20.33371875" size="2.54456875" layer="96"/>
+</instance>
+<instance part="S4" gate="G$1" x="68.58" y="5.08" smashed="yes">
+<attribute name="NAME" x="60.94906875" y="10.167290625" size="2.543640625" layer="95"/>
+<attribute name="VALUE" x="60.94628125" y="-2.55371875" size="2.54456875" layer="96"/>
+</instance>
+<instance part="S1" gate="G$1" x="68.58" y="22.86" smashed="yes">
+<attribute name="NAME" x="60.94906875" y="27.947290625" size="2.543640625" layer="95"/>
+<attribute name="VALUE" x="60.94628125" y="15.22628125" size="2.54456875" layer="96"/>
 </instance>
 </instances>
@@
 </segment>
 <segment>
-<pinref part="S1" gate="G$1" pin="1"/>
-<pinref part="S2" gate="G$1" pin="1"/>
-<wire x1="78.74" y1="22.86" x2="78.74" y2="5.08" width="0.1524" layer="91"/>
-<pinref part="S3" gate="G$1" pin="1"/>
-<wire x1="78.74" y1="5.08" x2="78.74" y2="-12.7" width="0.1524" layer="91"/>
+<pinref part="GND14" gate="1" pin="GND"/>
+<wire x1="78.74" y1="-33.02" x2="78.74" y2="-38.1" width="0.1524" layer="91"/>
+<pinref part="S2" gate="G$1" pin="SHIELD"/>
+<wire x1="78.74" y1="22.86" x2="78.74" y2="21.6662" width="0.1524" layer="91"/>
+<pinref part="S1" gate="G$1" pin="2"/>
+<pinref part="S4" gate="G$1" pin="2"/>
+<wire x1="78.74" y1="20.32" x2="78.74" y2="5.08" width="0.1524" layer="91"/>
+<pinref part="S1" gate="G$1" pin="SHIELD"/>
+<wire x1="78.74" y1="22.86" x2="78.74" y2="20.32" width="0.1524" layer="91"/>
+<junction x="78.74" y="22.86"/>
+<junction x="78.74" y="20.32"/>
+<pinref part="S3" gate="G$1" pin="2"/>
+<wire x1="78.74" y1="2.54" x2="78.74" y2="-12.7" width="0.1524" layer="91"/>
+<pinref part="S4" gate="G$1" pin="SHIELD"/>
+<wire x1="78.74" y1="5.08" x2="78.74" y2="2.54" width="0.1524" layer="91"/>
 <junction x="78.74" y="5.08"/>
-<pinref part="S4" gate="G$1" pin="1"/>
-<wire x1="78.74" y1="-12.7" x2="78.74" y2="-30.48" width="0.1524" layer="91"/>
+<junction x="78.74" y="2.54"/>
+<pinref part="S2" gate="G$1" pin="2"/>
+<wire x1="78.74" y1="-15.24" x2="78.74" y2="-30.48" width="0.1524" layer="91"/>
+<pinref part="S3" gate="G$1" pin="SHIELD"/>
+<wire x1="78.74" y1="-12.7" x2="78.74" y2="-15.24" width="0.1524" layer="91"/>
 <junction x="78.74" y="-12.7"/>
-<wire x1="78.74" y1="-30.48" x2="78.74" y2="-38.1" width="0.1524" layer="91"/>
+<junction x="78.74" y="-15.24"/>
+<wire x1="78.74" y1="-30.48" x2="78.74" y2="-33.02" width="0.1524" layer="91"/>
 <junction x="78.74" y="-30.48"/>
-<pinref part="GND14" gate="1" pin="GND"/>
+<junction x="78.74" y="-33.02"/>
 </segment>
 <segment>
@@
 <net name="SW1" class="0">
 <segment>
-<pinref part="S1" gate="G$1" pin="2"/>
 <pinref part="R32" gate="G$1" pin="1"/>
-<wire x1="53.34" y1="22.86" x2="50.8" y2="22.86" width="0.1524" layer="91"/>
+<wire x1="58.42" y1="22.86" x2="50.8" y2="22.86" width="0.1524" layer="91"/>
 <wire x1="50.8" y1="22.86" x2="50.8" y2="25.4" width="0.1524" layer="91"/>
 <wire x1="50.8" y1="22.86" x2="27.94" y2="22.86" width="0.1524" layer="91"/>
 <junction x="50.8" y="22.86"/>
 <label x="27.94" y="22.86" size="1.778" layer="95" rot="R180" xref="yes"/>
+<pinref part="S1" gate="G$1" pin="1"/>
 </segment>
 <segment>
@@
 <net name="SW2" class="0">
 <segment>
-<pinref part="S2" gate="G$1" pin="2"/>
 <pinref part="R33" gate="G$1" pin="1"/>
-<wire x1="53.34" y1="5.08" x2="45.72" y2="5.08" width="0.1524" layer="91"/>
+<wire x1="58.42" y1="5.08" x2="45.72" y2="5.08" width="0.1524" layer="91"/>
 <wire x1="45.72" y1="5.08" x2="45.72" y2="7.62" width="0.1524" layer="91"/>
 <wire x1="45.72" y1="5.08" x2="27.94" y2="5.08" width="0.1524" layer="91"/>
 <junction x="45.72" y="5.08"/>
 <label x="27.94" y="5.08" size="1.778" layer="95" rot="R180" xref="yes"/>
+<pinref part="S4" gate="G$1" pin="1"/>
 </segment>
 <segment>
@@
 <net name="SW3" class="0">
 <segment>
-<pinref part="S3" gate="G$1" pin="2"/>
 <pinref part="R34" gate="G$1" pin="1"/>
-<wire x1="53.34" y1="-12.7" x2="40.64" y2="-12.7" width="0.1524" layer="91"/>
+<wire x1="58.42" y1="-12.7" x2="40.64" y2="-12.7" width="0.1524" layer="91"/>
 <wire x1="40.64" y1="-12.7" x2="40.64" y2="-10.16" width="0.1524" layer="91"/>
 <wire x1="40.64" y1="-12.7" x2="27.94" y2="-12.7" width="0.1524" layer="91"/>
 <junction x="40.64" y="-12.7"/>
 <label x="27.94" y="-12.7" size="1.778" layer="95" rot="R180" xref="yes"/>
+<pinref part="S3" gate="G$1" pin="1"/>
 </segment>
 <segment>
@@
 <net name="SW4" class="0">
 <segment>
-<pinref part="S4" gate="G$1" pin="2"/>
 <pinref part="R35" gate="G$1" pin="1"/>
-<wire x1="53.34" y1="-30.48" x2="35.56" y2="-30.48" width="0.1524" layer="91"/>
+<wire x1="58.42" y1="-30.48" x2="35.56" y2="-30.48" width="0.1524" layer="91"/>
 <wire x1="35.56" y1="-30.48" x2="35.56" y2="-27.94" width="0.1524" layer="91"/>
 <wire x1="35.56" y1="-30.48" x2="27.94" y2="-30.48" width="0.1524" layer="91"/>
 <junction x="35.56" y="-30.48"/>
 <label x="27.94" y="-30.48" size="1.778" layer="95" rot="R180" xref="yes"/>
-</segment>
-<segment>
+<pinref part="S2" gate="G$1" pin="1"/>
+</segment>
+<segment>

Commit message: cs_v2_macrofab_sdc_version
Parts:
- removed J9: 47352-1001, 47352-1001:47352-1001
- added SD1: MF-MICROSD, MF_Connectors:SD_CARD_SLOT_MICRO_RIGHT
Connections:
- removed net N$19: J9.DATA1
- removed net N$45: J9.DATA2
- net 3V3_SDC: now also SD1.3.3V; no longer J9.VDD
- net GND: now also SD1.GND; no longer J9.SHIELD, J9.VSS
- net SD_CLK: now also SD1.SCLK; no longer J9.CLK
- net SD_CS: now also SD1.CS; no longer J9.CD/DATA3
- net SD_MISO: now also SD1.D0; no longer J9.DATA0
- net SD_MOSI: now also SD1.DI; no longer J9.CMD
Changed lines of the file:
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@@
 <part name="C8" library="SparkFun-Capacitors" deviceset="4.7PF" device="-0603-50V-5%" package3d_urn="urn:adsk.eagle:package:23616/2" value="10uF"/>
 <part name="C38" library="SparkFun-Capacitors" deviceset="4.7PF" device="-0603-50V-5%" package3d_urn="urn:adsk.eagle:package:23616/2" value="10uF"/>
-<part name="J9" library="47352-1001" deviceset="47352-1001" device="" package3d_urn="urn:adsk.eagle:package:16346114/2"/>
-<part name="GND19" library="supply1" library_urn="urn:adsk.eagle:library:371" deviceset="GND" device=""/>
 <part name="R16" library="MF_Passives" deviceset="RESISTOR" device="_0603" package3d_urn="urn:adsk.eagle:package:16347927/2" value="10K"/>
 <part name="C20" library="MF_Passives" deviceset="CAPACITOR_NP" device="_0603" package3d_urn="urn:adsk.eagle:package:16347923/3" value="1uF"/>
@@
 <part name="S4" library="EVQ-P4HB3B" deviceset="EVQ-P4HB3B" device="" override_package3d_urn="urn:adsk.eagle:package:16346036/2" override_package_urn="urn:adsk.eagle:footprint:16346037/1" override_locally_modified="yes"/>
 <part name="S1" library="EVQ-P4HB3B" deviceset="EVQ-P4HB3B" device="" override_package3d_urn="urn:adsk.eagle:package:16346036/2" override_package_urn="urn:adsk.eagle:footprint:16346037/1" override_locally_modified="yes"/>
+<part name="SD1" library="MF_Connectors" deviceset="SD_CARD_SLOT" device="_MICRO_RIGHT" package3d_urn="urn:adsk.eagle:package:9948224/2" value="MF-MICROSD"/>
 </parts>
 <sheets>
@@
 <attribute name="VALUE" x="94.996" y="197.739" size="1.778" layer="96" font="vector" rot="R180"/>
 </instance>
-<instance part="J9" gate="G$1" x="388.62" y="154.94" smashed="yes">
-<attribute name="NAME" x="381" y="170.942" size="1.778" layer="95"/>
-<attribute name="VALUE" x="381" y="137.16" size="1.778" layer="96"/>
-</instance>
-<instance part="GND19" gate="1" x="375.92" y="139.7" smashed="yes">
-<attribute name="VALUE" x="373.38" y="137.16" size="1.778" layer="96"/>
-</instance>
 <instance part="U6" gate="G$1" x="388.62" y="106.68" smashed="yes">
 <attribute name="NAME" x="378.46" y="125.222" size="1.778" layer="95"/>
@@
 <attribute name="NAME" x="60.94906875" y="27.947290625" size="2.543640625" layer="95"/>
 <attribute name="VALUE" x="60.94628125" y="15.22628125" size="2.54456875" layer="96"/>
+</instance>
+<instance part="SD1" gate="G$1" x="347.98" y="170.18" smashed="yes">
+<attribute name="NAME" x="347.98" y="173.99" size="1.016" layer="95" font="vector" align="top-left"/>
+<attribute name="VALUE" x="347.98" y="171.45" size="1.016" layer="96" font="vector"/>
 </instance>
 </instances>
@@
 <wire x1="342.9" y1="144.78" x2="342.9" y2="142.24" width="0.1524" layer="91"/>
 <pinref part="GND12" gate="1" pin="GND"/>
+<pinref part="SD1" gate="G$1" pin="GND"/>
 </segment>
 <segment>
@@
 </segment>
 <segment>
-<pinref part="J9" gate="G$1" pin="VSS"/>
-<pinref part="J9" gate="G$1" pin="SHIELD"/>
-<wire x1="375.92" y1="147.32" x2="375.92" y2="142.24" width="0.1524" layer="91"/>
-<pinref part="GND19" gate="1" pin="GND"/>
-<junction x="375.92" y="142.24"/>
-</segment>
-<segment>
 <pinref part="U6" gate="G$1" pin="GND"/>
 <pinref part="U6" gate="G$1" pin="GNDIO"/>
@@
 <wire x1="325.12" y1="165.1" x2="325.12" y2="170.18" width="0.1524" layer="91"/>
 <label x="325.12" y="165.1" size="1.27" layer="95" rot="R270" xref="yes"/>
+<pinref part="SD1" gate="G$1" pin="CS"/>
 </segment>
 <segment>
@@
 <wire x1="71.12" y1="147.32" x2="73.66" y2="147.32" width="0.1524" layer="91"/>
 <label x="73.66" y="147.32" size="1.27" layer="95" xref="yes"/>
-</segment>
-<segment>
-<pinref part="J9" gate="G$1" pin="CD/DATA3"/>
-<wire x1="375.92" y1="160.02" x2="373.38" y2="160.02" width="0.1524" layer="91"/>
-<label x="373.38" y="160.02" size="1.016" layer="95" rot="R180" xref="yes"/>
 </segment>
 </net>
@@
 <wire x1="317.5" y1="162.56" x2="317.5" y2="170.18" width="0.1524" layer="91"/>
 <label x="317.5" y="162.56" size="1.27" layer="95" rot="R270" xref="yes"/>
+<pinref part="SD1" gate="G$1" pin="DI"/>
 </segment>
 <segment>
@@
 <wire x1="30.48" y1="144.78" x2="27.94" y2="144.78" width="0.1524" layer="91"/>
 <label x="27.94" y="144.78" size="1.27" layer="95" rot="R180" xref="yes"/>
-</segment>
-<segment>
-<pinref part="J9" gate="G$1" pin="CMD"/>
-<wire x1="375.92" y1="157.48" x2="373.38" y2="157.48" width="0.1524" layer="91"/>
-<label x="373.38" y="157.48" size="1.016" layer="95" rot="R180" xref="yes"/>
 </segment>
 </net>
@@
 <wire x1="309.88" y1="160.02" x2="309.88" y2="170.18" width="0.1524" layer="91"/>
 <label x="309.88" y="160.02" size="1.27" layer="95" rot="R270" xref="yes"/>
+<pinref part="SD1" gate="G$1" pin="SCLK"/>
 </segment>
 <segment>
@@
 <wire x1="30.48" y1="134.62" x2="27.94" y2="134.62" width="0.1524" layer="91"/>
 <label x="27.94" y="134.62" size="1.27" layer="95" rot="R180" xref="yes"/>
-</segment>
-<segment>
-<pinref part="J9" gate="G$1" pin="CLK"/>
-<wire x1="375.92" y1="154.94" x2="373.38" y2="154.94" width="0.1524" layer="91"/>
-<label x="373.38" y="154.94" size="1.016" layer="95" rot="R180" xref="yes"/>
 </segment>
 </net>
@@
 <label x="302.26" y="157.48" size="1.27" layer="95" rot="R270" xref="yes"/>
 <pinref part="R43" gate="G$1" pin="1"/>
+<pinref part="SD1" gate="G$1" pin="D0"/>
 </segment>
 <segment>
@@
 <wire x1="30.48" y1="137.16" x2="27.94" y2="137.16" width="0.1524" layer="91"/>
 <label x="27.94" y="137.16" size="1.27" layer="95" rot="R180" xref="yes"/>
-</segment>
-<segment>
-<pinref part="J9" gate="G$1" pin="DATA0"/>
-<wire x1="375.92" y1="167.64" x2="373.38" y2="167.64" width="0.1524" layer="91"/>
-<label x="373.38" y="167.64" size="1.016" layer="95" rot="R180" xref="yes"/>
 </segment>
 </net>
@@
 <pinref part="R43" gate="G$1" pin="2"/>
 <junction x="302.26" y="180.34"/>
-</segment>
-<segment>
-<pinref part="J9" gate="G$1" pin="VDD"/>
-<wire x1="375.92" y1="149.86" x2="373.38" y2="149.86" width="0.1524" layer="91"/>
-<label x="373.38" y="149.86" size="1.016" layer="95" rot="R180" xref="yes"/>
+<pinref part="SD1" gate="G$1" pin="3.3V"/>
 </segment>
 </net>
@@
 </segment>
 </net>
-<net name="N$45" class="0">
-<segment>
-<pinref part="J9" gate="G$1" pin="DATA2"/>
-<wire x1="375.92" y1="162.56" x2="373.38" y2="162.56" width="0.1524" layer="91"/>
-</segment>
-</net>
-<net name="N$19" class="0">
-<segment>
-<pinref part="J9" gate="G$1" pin="DATA1"/>
-<wire x1="375.92" y1="165.1" x2="373.38" y2="165.1" width="0.1524" layer="91"/>
-</segment>
-</net>

Commit message: reassigned input-only pins
Connections:
- net ACCL1 renamed GPIO_EXT
- removed net ACCL2: ESP32-PICO-D4.IO32, U6.INT1
- removed net MAGDRDY: ESP32-PICO-D4.IO34, U$5.EXTCOMIN
- new net BMX_INT: ESP32-PICO-D4.IO34, U6.INT1
- new net LCD_EXTCOMM: ESP32-PICO-D4.IO32, U$5.EXTCOMIN
Changed lines of the file:
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@@
 </segment>
 </net>
-<net name="ACCL1" class="0">
+<net name="GPIO_EXT" class="0">
 <segment>
 <pinref part="ESP32-PICO-D4" gate="G$1" pin="IO33"/>
@@
 </segment>
 </net>
-<net name="ACCL2" class="0">
+<net name="LCD_EXTCOMM" class="0">
 <segment>
 <pinref part="ESP32-PICO-D4" gate="G$1" pin="IO32"/>
@@
 </segment>
 <segment>
-<pinref part="U6" gate="G$1" pin="INT1"/>
-<wire x1="373.38" y1="101.6" x2="370.84" y2="101.6" width="0.1524" layer="91"/>
-<label x="370.84" y="101.6" size="1.27" layer="95" rot="R180" xref="yes"/>
-</segment>
-</net>
-<net name="MAGDRDY" class="0">
-<segment>
-<pinref part="ESP32-PICO-D4" gate="G$1" pin="IO34"/>
-<wire x1="30.48" y1="162.56" x2="27.94" y2="162.56" width="0.1524" layer="91"/>
-<label x="27.94" y="162.56" size="1.27" layer="95" rot="R180" xref="yes"/>
-</segment>
-<segment>
 <pinref part="U$5" gate="G$1" pin="EXTCOMIN"/>
-<wire x1="322.58" y1="35.56" x2="345.44" y2="35.56" width="0.1524" layer="91"/>
-<label x="322.58" y="35.56" size="1.27" layer="95" rot="R180" xref="yes"/>
+<wire x1="345.44" y1="35.56" x2="342.9" y2="35.56" width="0.1524" layer="91"/>
+<label x="342.9" y="35.56" size="1.778" layer="95" rot="R180" xref="yes"/>
 </segment>
 </net>
@@
 </segment>
 </net>
+<net name="BMX_INT" class="0">
+<segment>
+<pinref part="U6" gate="G$1" pin="INT1"/>
+<wire x1="373.38" y1="101.6" x2="370.84" y2="101.6" width="0.1524" layer="91"/>
+<label x="370.84" y="101.6" size="1.27" layer="95" rot="R180" xref="yes"/>
+</segment>
+<segment>
+<pinref part="ESP32-PICO-D4" gate="G$1" pin="IO34"/>
+<wire x1="30.48" y1="162.56" x2="27.94" y2="162.56" width="0.1524" layer="91"/>
+<label x="27.94" y="162.56" size="1.27" layer="95" rot="R180" xref="yes"/>
+</segment>
+</net>
